File: eater-deluxe.kicad_pcb (KiCad board)
At the start: 2 copper layers, 214.2 x 149.5 mm, 39 parts, among them J1 PJ-202A, J2 DE9_Socket, SW1 RESET, U1 6502, U2 W65C22NxP, U3 W65C51NxP, U4 28C256, U5 HM62256BLP, U6 CD74HC00E, U7 MAX232, U8 LCD Module Connector, X1 MXO45-3C-1M000000, Y1 1.8432MHz

Commit message: revision 1.0 completely finished
Signed-off-by: Lucy <user@domain.tld>
Parts:
- H1, H2, H3, H4: value MountingHole -> M3
Other:
- board text added: "${TITLE} Revision ${REVISION} ${ISSUE_DATE} ${COMMENT1}"
- board text added: "CC-BY"
